File: src_files/power supply.kicad_sch (KiCad schematic)
At the start: 17 parts

Commit message: updated footprint assignment
Parts:
- added TP1: +50V, TestPoint:TestPoint_Pad_D1.0mm, symbol Connector:TestPoint
- added TP2: -50V, TestPoint:TestPoint_Pad_D1.0mm, symbol Connector:TestPoint
- C10, C11, C12, C13, C14, C15: renamed from C?; footprint (none) -> Capacitor_SMD:C_0603_1608Metric_Pad1.08x0.95mm_HandSolder
- C16: renamed from C?; footprint (none) -> Capacitor_SMD:C_1206_3216Metric_Pad1.33x1.80mm_HandSolder
- C17: renamed from C?; value 4700pF -> 4700pF_250V; footprint (none) -> Capacitor_SMD:C_0805_2012Metric_Pad1.18x1.45mm_HandSolder
- R3, R4, R5, R6: renamed from R?; footprint (none) -> Resistor_SMD:R_0603_1608Metric_Pad0.98x0.95mm_HandSolder
- U3: renamed from U?; footprint (none) -> Package_TO_SOT_SMD:SOT-223-3_TabPin2
- gave numbers to parts that had none: 4
Connections:
- net +50V: now also TP1.1
- net -50V: now also TP2.1
